File: hardware/CAN TOF.brd (EAGLE design)
At the start: 33 x 43.2 mm, 35 parts, among them Q1 8MHz, T2 BSS138, U1 ATMEGA328P_TQFP, U2 MCP2515, U3 MCP2551

Commit message: switching to atmel studio. also there are proj files here. sue me.
Parts:
- added C8, C9: 20pF, rcl:C0402
- added Q2: 16MHz, crystal:CTS406
Connections:
- new net N$12: C8.1, Q2.1, U1.8
- new net N$13: C9.1, Q2.3, U1.7
- net GND: now also C8.2, C9.2
Changed lines of the file:
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@@
 <attribute name="VALUE" x="27.305" y="12.065" size="1.27" layer="27" rot="R270"/>
+</element>
+<element name="Q2" library="crystal" library_urn="urn:adsk.eagle:library:204" package="CTS406" package3d_urn="urn:adsk.eagle:package:12089/1" value="16MHz" x="3.81" y="-5.08" smashed="yes">
+<attribute name="MF" value="" x="-5.08" y="5.08" size="1.778" layer="27" display="off"/>
+<attribute name="MPN" value="" x="-5.08" y="5.08" size="1.778" layer="27" display="off"/>
+<attribute name="NAME" x="1.27" y="-2.54" size="1.27" layer="25"/>
+<attribute name="OC_FARNELL" value="unknown" x="-5.08" y="5.08" size="1.778" layer="27" display="off"/>
+<attribute name="OC_NEWARK" value="unknown" x="-5.08" y="5.08" size="1.778" layer="27" display="off"/>
+<attribute name="VALUE" x="1.27" y="-8.89" size="1.27" layer="27"/>
+</element>
+<element name="C8" library="rcl" library_urn="urn:adsk.eagle:library:334" package="C0402" package3d_urn="urn:adsk.eagle:package:23626/2" value="20pF" x="1.27" y="-12.7" smashed="yes">
+<attribute name="NAME" x="0.635" y="-12.065" size="1.27" layer="25"/>
+<attribute name="SPICEPREFIX" value="C" x="-6.35" y="-3.81" size="1.778" layer="27" display="off"/>
+<attribute name="VALUE" x="0.635" y="-14.605" size="1.27" layer="27"/>
+</element>
+<element name="C9" library="rcl" library_urn="urn:adsk.eagle:library:334" package="C0402" package3d_urn="urn:adsk.eagle:package:23626/2" value="20pF" x="1.27" y="-17.78" smashed="yes">
+<attribute name="NAME" x="0.635" y="-17.145" size="1.27" layer="25"/>
+<attribute name="SPICEPREFIX" value="C" x="-6.35" y="-8.89" size="1.778" layer="27" display="off"/>
+<attribute name="VALUE" x="0.635" y="-19.685" size="1.27" layer="27"/>
 </element>
 </elements>
@@
 <vertex x="33.02" y="0"/>
 </polygon>
+<contactref element="C8" pad="2"/>
+<contactref element="C9" pad="2"/>
+<wire x1="1.92" y1="-12.7" x2="1.92" y2="-17.78" width="0" layer="19" extent="1-1"/>
+<wire x1="7.62" y1="4.445" x2="1.92" y2="-12.7" width="0" layer="19" extent="1-16"/>
 </signal>
 <signal name="INT0">
@@
 <via x="3.96875" y="11.90625" extent="1-16" drill="0.35"/>
 </signal>
+<signal name="N$12">
+<contactref element="C8" pad="1"/>
+<contactref element="Q2" pad="1"/>
+<contactref element="U1" pad="8"/>
+<wire x1="1.61" y1="-6.28" x2="14.4526" y2="32.76" width="0" layer="19" extent="1-16"/>
+<wire x1="0.62" y1="-12.7" x2="1.61" y2="-6.28" width="0" layer="19" extent="1-1"/>
+</signal>
+<signal name="N$13">
+<contactref element="C9" pad="1"/>
+<contactref element="Q2" pad="3"/>
+<contactref element="U1" pad="7"/>
+<wire x1="6.01" y1="-3.88" x2="14.4526" y2="33.56" width="0" layer="19" extent="1-16"/>
+<wire x1="0.62" y1="-17.78" x2="6.01" y2="-3.88" width="0" layer="19" extent="1-1"/>
+</signal>
 </signals>

Commit message: switching to 20Mhz crystal...
Parts:
- removed C8, C9: 20pF, rcl:C0402
- removed Q2: 16MHz, crystal:CTS406
- Q1: value 8MHz -> 20MHz
Connections:
- removed net N$12: C8.1, Q2.1, U1.8
- removed net N$13: C9.1, Q2.3, U1.7
- net GND: no longer C8.2, C9.2
Changed lines of the file:
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@@
 <attribute name="VALUE" x="14.605" y="36.83" size="1.27" layer="27"/>
 </element>
-<element name="Q1" library="crystal" library_urn="urn:adsk.eagle:library:204" package="CTS406" package3d_urn="urn:adsk.eagle:package:12089/1" value="8MHz" x="27.94" y="31.75" smashed="yes">
+<element name="Q1" library="crystal" library_urn="urn:adsk.eagle:library:204" package="CTS406" package3d_urn="urn:adsk.eagle:package:12089/1" value="20MHz" x="27.94" y="31.75" smashed="yes">
 <attribute name="MF" value="" x="3.81" y="7.62" size="1.778" layer="27" display="off"/>
 <attribute name="MPN" value="" x="3.81" y="7.62" size="1.778" layer="27" display="off"/>
@@
 <attribute name="SPICEPREFIX" value="R" x="29.845" y="11.43" size="1.778" layer="27" rot="R270" display="off"/>
 <attribute name="VALUE" x="27.305" y="12.065" size="1.27" layer="27" rot="R270"/>
-</element>
-<element name="Q2" library="crystal" library_urn="urn:adsk.eagle:library:204" package="CTS406" package3d_urn="urn:adsk.eagle:package:12089/1" value="16MHz" x="3.81" y="-5.08" smashed="yes">
-<attribute name="MF" value="" x="-5.08" y="5.08" size="1.778" layer="27" display="off"/>
-<attribute name="MPN" value="" x="-5.08" y="5.08" size="1.778" layer="27" display="off"/>
-<attribute name="NAME" x="1.27" y="-2.54" size="1.27" layer="25"/>
-<attribute name="OC_FARNELL" value="unknown" x="-5.08" y="5.08" size="1.778" layer="27" display="off"/>
-<attribute name="OC_NEWARK" value="unknown" x="-5.08" y="5.08" size="1.778" layer="27" display="off"/>
-<attribute name="VALUE" x="1.27" y="-8.89" size="1.27" layer="27"/>
-</element>
-<element name="C8" library="rcl" library_urn="urn:adsk.eagle:library:334" package="C0402" package3d_urn="urn:adsk.eagle:package:23626/2" value="20pF" x="1.27" y="-12.7" smashed="yes">
-<attribute name="NAME" x="0.635" y="-12.065" size="1.27" layer="25"/>
-<attribute name="SPICEPREFIX" value="C" x="-6.35" y="-3.81" size="1.778" layer="27" display="off"/>
-<attribute name="VALUE" x="0.635" y="-14.605" size="1.27" layer="27"/>
-</element>
-<element name="C9" library="rcl" library_urn="urn:adsk.eagle:library:334" package="C0402" package3d_urn="urn:adsk.eagle:package:23626/2" value="20pF" x="1.27" y="-17.78" smashed="yes">
-<attribute name="NAME" x="0.635" y="-17.145" size="1.27" layer="25"/>
-<attribute name="SPICEPREFIX" value="C" x="-6.35" y="-8.89" size="1.778" layer="27" display="off"/>
-<attribute name="VALUE" x="0.635" y="-19.685" size="1.27" layer="27"/>
 </element>
 </elements>
@@
 <vertex x="33.02" y="0"/>
 </polygon>
-<contactref element="C8" pad="2"/>
-<contactref element="C9" pad="2"/>
-<wire x1="1.92" y1="-12.7" x2="1.92" y2="-17.78" width="0" layer="19" extent="1-1"/>
-<wire x1="7.62" y1="4.445" x2="1.92" y2="-12.7" width="0" layer="19" extent="1-16"/>
 </signal>
 <signal name="INT0">
@@
 <via x="3.96875" y="11.90625" extent="1-16" drill="0.35"/>
 </signal>
-<signal name="N$12">
-<contactref element="C8" pad="1"/>
-<contactref element="Q2" pad="1"/>
-<contactref element="U1" pad="8"/>
-<wire x1="1.61" y1="-6.28" x2="14.4526" y2="32.76" width="0" layer="19" extent="1-16"/>
-<wire x1="0.62" y1="-12.7" x2="1.61" y2="-6.28" width="0" layer="19" extent="1-1"/>
-</signal>
-<signal name="N$13">
-<contactref element="C9" pad="1"/>
-<contactref element="Q2" pad="3"/>
-<contactref element="U1" pad="7"/>
-<wire x1="6.01" y1="-3.88" x2="14.4526" y2="33.56" width="0" layer="19" extent="1-16"/>
-<wire x1="0.62" y1="-17.78" x2="6.01" y2="-3.88" width="0" layer="19" extent="1-1"/>
-</signal>
 </signals>
